File: pcb/pcb.kicad_sch (KiCad schematic)
At the start: 18 parts, among them J1 Power, Q1 Q_NPN_BCE, SW1 START, SW2 RESET, U1 PIC16F18346-P, U2 74HC595, U3 SCORE 1, U4 SCORE 2

Commit message: Finish v.1 schematic
Parts:
- removed U4: SCORE 2, Display_7Segment:Sx39-1xxxxx, symbol Display_Character:SC39-11GWA
- added C5, C6, C7: 100nF, symbol Device:C_Small
- added C8: 10uF, symbol Device:C_Small
- added R10, R12, R14, R16, R18, R4, R6, R8: 330, symbol Device:R
- added R11, R13, R15, R17, R3, R5, R7, R9: 330Ω, symbol Device:R
- added R19: 10kΩ, symbol Device:R
- added TP1, TP2, TP3, TP4, TP5, TP6: TestPoint, symbol Connector:TestPoint
- added U4: 74HC595, symbol 74xx:74HC595
- added U5: SCORE 1, Display_7Segment:Sx39-1xxxxx, symbol Display_Character:SC39-11GWA
- U6: renamed from SSD1306; value OLED -> SSD1306
Connections:
- net +3.3V: now also U2.10 (~{SRCLR}), U2.16 (VCC), C5.1, C6.1, C7.1, C8.1, R19.1, TP4.1, U4.10 (~{SRCLR}), U4.16 (VCC)
- net BUZZER: now also U1.13 (RB4); no longer U1.14 (RC2)
- net Earth: now also U1.4 (RA3/~{MCLR}/VPP), U2.13 (~{OE}), U2.8 (GND), U3.3 (CC), U3.8 (CC), C5.2, C6.2, C7.2, C8.2, R19.2, TP3.1, TP5.1, U4.13 (~{OE}), U4.8 (GND), U5.3 (CC), U5.8 (CC)
- net P1: now also U1.12 (RB5); no longer U1.16 (RC0)
- net P2: now also U1.11 (RB6); no longer U1.15 (RC1)
- net at U3.1 (G): now also R9.2
- net at U3.10 (A): now also R3.2
- net at U3.2 (F): now also R8.2
- net at U3.4 (E): now also R7.2
- net at U3.5 (D): now also R6.2
- net at U3.6 (DP): now also R10.2
- net at U3.7 (C): now also R5.2
- net at U3.9 (B): now also R4.2
- net at U2.1 (QB): now also R4.1
- net SRCLK: now reaches U2.11 (SRCLK)
- net SRCLK: now also U1.15 (RC1), U4.11 (SRCLK)
- net RCLK: now reaches U2.12 (RCLK)
- net RCLK: now also U1.14 (RC2), U4.12 (RCLK)
- net SER: now reaches U2.14 (SER)
- net SER: now also U1.16 (RC0)
- net at U2.15 (QA): now also R3.1
- net at U2.2 (QC): now also R5.1
- net at U2.3 (QD): now also R6.1
- net at U2.4 (QE): now also R7.1
- net at U2.5 (QF): now also R8.1
- net at U2.6 (QG): now also R9.1
- net at U2.7 (QH): now also R10.1
- net at U2.9 (QH'): now also U4.14 (SER)
- net ICSPCLK: now reaches U1.18 (RA1/ICSPCLK)
- net ICSPCLK: now also TP2.1
- net ISCPDAT: now reaches U1.19 (RA0/ICSPDAT)
- net ISCPDAT: now also TP1.1
- new net: R12.1, U4.1 (QB)
- new net: R12.2, U5.9 (B)
- new net: R17.1, U4.6 (QG)
- new net: R17.2, U5.1 (G)
- new net: R11.1, U4.15 (QA)
- new net: R11.2, U5.10 (A)
- new net: R18.1, U4.7 (QH)
- new net: R18.2, U5.6 (DP)
- new net: R16.2, U5.2 (F)
- new net: R15.2, U5.4 (E)
- new net: R14.2, U5.5 (D)
- new net: R13.2, U5.7 (C)
- new net: R16.1, U4.5 (QF)
- new net: R13.1, U4.2 (QC)
- new net: R14.1, U4.3 (QD)
- new net: R15.1, U4.4 (QE)
- no-connect marks 0 -> 1
Other:
- note added: "PIC"
- note added: "Score Displays"
- moved on the sheet: BZ1, C1, C2, C3, C4, J1, Paddle1, Paddle2, Q1, R1, R2, SW1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

Commit message: Breadboarding and added transistor for seven segment displays
Parts:
- added Q2, Q3: Q_NPN_BCE, symbol Transistor_BJT:Q_NPN_BCE
Connections:
- net BUZZER: now also U1.17 (RA2); no longer U1.13 (RB4)
- net Earth: now also Q2.3 (E), Q3.3 (E); no longer U3.3 (CC), U3.8 (CC), U5.3 (CC), U5.8 (CC)
- net P1: now also U1.3 (RA4); no longer U1.12 (RB5)
- net P2: now also U1.2 (RA5); no longer U1.11 (RB6)
- net RESET: now also U1.12 (RB5); no longer U1.2 (RA5)
- net START: now also U1.13 (RB4); no longer U1.3 (RA4)
- net EN2: now reaches U1.10 (RB7)
- net EN2: now also Q3.1 (B)
- new net: Q2.2 (C), U3.3 (CC), U3.8 (CC)
- new net: Q3.2 (C), U5.3 (CC), U5.8 (CC)
- new net EN1: Q2.1 (B), U1.11 (RB6)
Other:
- moved on the sheet: C6, C7, R10, R11, R12, R13, R14, R15, R16, R17, R18, R3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

Commit message: Read potentiometers & move WAIT to BANK0
Parts:
- removed Q2, Q3: Q_NPN_BCE, symbol Transistor_BJT:Q_NPN_BCE
Connections:
- net EN1 is gone; now on net RESET: U1.11 (RB6)
- net BUZZER: now also U1.13 (RB4); no longer U1.17 (RA2)
- net EN2: no longer U1.10 (RB7)
- net Earth: now also U3.3 (CC), U3.8 (CC), U5.3 (CC), U5.8 (CC)
- net RESET: no longer U1.12 (RB5)
- net START: now also U1.12 (RB5); no longer U1.13 (RB4)

Commit message: Setup PPS
Other:
- note added: "(SCK)"
- note added: "(SDA)"
Changed lines of the file:
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@@
+		)
+	)
+	(text "(SCK)\n"
+		(exclude_from_sim no)
+		(at 188.722 75.438 0)
+		(effects
+			(font
+				(size 1.27 1.27)
+			)
+		)
+	)
+	(text "(SDA)"
+		(exclude_from_sim no)
+		(at 188.722 77.978 0)
+		(effects
+			(font
+				(size 1.27 1.27)
+			)
 		)
 	)

Commit message: Add ball update subroutines
Parts:
- added R20: 1kΩ, symbol Device:R
Connections:
- net BUZZER: now also R20.1; no longer Q1.1 (B)
- new net: Q1.1 (B), R20.2
Other:
- company: (none) -> tecknet-gg, jeevan hatti
- title: (none) -> asm-pong
- moved on the sheet: BZ1, C1, C2, C3, C4, C5, C6, C7, C8, J1, Paddle1, Paddle2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
