File: pcb/pcb.kicad_pcb (KiCad board)
At the start: 2 copper layers, 44 parts, among them J1 ICSP, J2 Debug 1, J3 Debug 2, P1 Power, Q1 Q_NPN_BCE, SW1 START, SW2 RESET, U1 PIC16F18346-P, U2 74HC595, U3 SCORE 1, U4 74HC595, U5 SCORE 2, U6 SSD1306

Commit message: Layout PCB
Parts:
- added D1: D_Small, Diode_THT:D_DO-35_SOD27_P7.62mm_Horizontal, F.Cu at (155.4, 102.5)
- Paddle 1: renamed from Paddle1
- Paddle 2: renamed from Paddle2
- R10: value 330 -> 330Ω
- U2, U4: footprint Package_DIP:DIP-16_W7.62mm_LongPads -> Package_DIP:DIP-16_W7.62mm_Socket_LongPads
- moved R2 135.6 mm to (174.5, 119.1), turned to 90 degrees
- moved R18 126.4 mm to (192.0, 83.0), turned to 90 degrees
- moved R19 126.1 mm to (189.0, 114.6), turned to 90 degrees
- moved R16 123.5 mm to (189.0, 83.0), turned to 90 degrees
- moved R17 120.4 mm to (186.0, 83.0), turned to 90 degrees
- moved R15 117.8 mm to (183.0, 83.0), turned to 90 degrees
- moved Paddle 2 115.8 mm to (184.0, 128.9), turned to -90 degrees
- moved R14 104.2 mm to (169.8, 66.5)
- moved R11 104.2 mm to (169.8, 57.5)
- moved R13 104.2 mm to (169.8, 63.5)
- moved R12 104.2 mm to (169.8, 60.5)
- moved R1 96.4 mm to (125.5, 119.0), turned to 90 degrees
- moved U1 96.3 mm to (138.4, 140.0), turned to 90 degrees
- moved J1 87.7 mm to (195.0, 107.8)
- moved C2 86.8 mm to (167.5, 129.0)
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Connections:
- Paddle 2 pad 1: Earth -> +3.3V
- Paddle 2 pad 3: +3.3V -> Earth
Other:
- board outline added: 98.2 x 95.2 mm
- board text added: "330Ω"
- board text added: "OLED"
