File: pcb/pcb.kicad_pcb (KiCad board)
At the start: 2 copper layers, 98.2 x 95.2 mm, 45 parts, among them J1 ICSP, J2 Debug 1, J3 Debug 2, P1 Power, Q1 Q_NPN_BCE, SW1 START, SW2 RESET, U1 PIC16F18346-P, U2 74HC595, U3 SCORE 1, U4 74HC595, U5 SCORE 2, U6 SSD1306

Commit message: Route PCB
Parts:
- added C9: 1uF, Capacitor_THT:C_Radial_D4.0mm_H7.0mm_P1.50mm, F.Cu at (118.3, 110.0)
- added G***: LOGO, LOGO, B.Cu at (149.6, 69.7)
- added U7: MCP1700x-330xxTO, Package_TO_SOT_THT:TO-92_Inline, F.Cu at (111.5, 107.4)
- C8: value 10uF -> 1uF; footprint Capacitor_THT:C_Radial_D5.0mm_H11.0mm_P2.00mm -> Capacitor_THT:C_Radial_D4.0mm_H7.0mm_P1.50mm
- Q1: value Q_NPN_BCE -> 2N2222
- R10: value 330Ω -> 330
- R11, R3: value 330Ω -> 220Ω
- R20: value 1kΩ -> 1kΩ
- U1: value PIC16F18346-P -> PIC16F18346
- moved R16 31.8 mm to (169.9, 57.5), turned to 0 degrees
- moved R11 29.3 mm to (183.0, 83.7), turned to 90 degrees
- moved R12 28.2 mm to (186.0, 83.7), turned to 90 degrees
- moved R6 27.9 mm to (106.0, 83.6), turned to 90 degrees
- moved R13 27.8 mm to (189.0, 83.7), turned to 90 degrees
- moved R17 27.7 mm to (169.9, 60.5), turned to 0 degrees
- moved R15 23.5 mm to (169.9, 63.5), turned to 0 degrees
- moved C6 21.6 mm to (129.0, 97.5), turned to 180 degrees
- moved R10 21.5 mm to (128.1, 66.5), turned to 180 degrees
- moved U4 21.3 mm to (168.5, 76.0), turned to 0 degrees
- moved C7 17.7 mm to (175.0, 97.5), turned to 180 degrees
- moved U2 15.9 mm to (123.0, 76.0), turned to 0 degrees
- moved C1 14.3 mm to (115.5, 122.0)
- moved C2 13.9 mm to (179.5, 122.0)
- moved P1 12.2 mm to (115.5, 97.0)
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Connections:
- C8 pad 1: +3.3V -> VIN
- J3 pad 4: unconnected-(J3-Pin_4-Pad4) -> VIN
- P1 pad 1: +3.3V -> VIN
- P1 pad 2: unconnected-(P1-Pad2) -> Earth
- P1 pad 3: Earth -> unconnected-(P1-Pad3)
- Q1 pad 1: Net-(Q1-B) -> Earth
- Q1 pad 2: Net-(BZ1--) -> Net-(Q1-B)
- Q1 pad 3: Earth -> Net-(BZ1--)
- U1 pad 2: /P2 -> /P1
- U1 pad 3: /P1 -> /P2
Routing:
- net +3.3V: track 0.00 -> 335.9 mm
- net /RESET: track 0.00 -> 110.6 mm
- net /P2: track 0.00 -> 107.5 mm
- net /CS: track 0.00 -> 98.6 mm, vias 0 -> 4
- net /RCLK: track 0.00 -> 98.0 mm, vias 0 -> 9
- net /START: track 0.00 -> 96.0 mm
- net /D1: track 0.00 -> 95.6 mm, vias 0 -> 4
- net /D0: track 0.00 -> 92.6 mm, vias 0 -> 2
- net /DC: track 0.00 -> 90.7 mm, vias 0 -> 4
- net /SRCLK: track 0.00 -> 89.9 mm, vias 0 -> 6
- net /RES: track 0.00 -> 88.6 mm, vias 0 -> 2
- net /BUZZER: track 0.00 -> 81.4 mm, vias 0 -> 2
- net /MCLR/VPP: track 0.00 -> 71.2 mm, vias 0 -> 2
- net /ICSPDAT: track 0.00 -> 64.8 mm, vias 0 -> 3
- net /ICSPCLK: track 0.00 -> 63.1 mm, vias 0 -> 3
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- added copper zone on B.Cu, net Earth
- added copper zone on F.Cu, net Earth
Other:
- board text added: "220Ω"
- board text added: "asm-pong"
- board text added: "made by jeevan"
- board text added: "made by tecknet"
- board text added: "tecknet.dev"
- board text removed: "330Ω"

Commit message: Finish 3D model and render
Parts:
- added H1: MountingHole, MountingHole:MountingHole_2.2mm_M2, F.Cu at (194.5, 55.5)
- added H2: MountingHole, MountingHole:MountingHole_2.2mm_M2, F.Cu at (103.5, 55.5)
- added H3: MountingHole, MountingHole:MountingHole_2.2mm_M2, F.Cu at (103.5, 143.5)
- added H4: MountingHole, MountingHole:MountingHole_2.2mm_M2, F.Cu at (194.5, 143.5)
- Paddle1: renamed from Paddle 1
- Paddle2: renamed from Paddle 2
- R20: value 1kΩ -> 1kΩ
- U1: value PIC16F18346 -> PIC16F18346-P
