File: pcb/_autosave-pcb.kicad_pcb (KiCad board)
At the start: 2 copper layers, 98.2 x 95.2 mm, 45 parts, among them J1 ICSP, J2 Debug 1, J3 Debug 2, P1 Power, Q1 Q_NPN_BCE, SW1 START, SW2 RESET, U1 PIC16F18346-P, U2 74HC595, U3 SCORE 1, U4 74HC595, U5 SCORE 2, U6 SSD1306

Commit message: Hardware testing
Parts:
- Paddle1: renamed from Paddle 1
- Paddle2: renamed from Paddle 2
- Q1: value Q_NPN_BCE -> BC107
- R10: value 330Ω -> 330
- moved C6 21.6 mm to (129.0, 97.5), turned to 180 degrees
- moved U4 21.3 mm to (168.5, 76.0), turned to 0 degrees
- moved C7 17.7 mm to (175.0, 97.5), turned to 180 degrees
- moved U2 15.9 mm to (123.0, 76.0), turned to 0 degrees
- moved C1 14.3 mm to (115.5, 122.0)
- moved C2 13.9 mm to (179.5, 122.0)
- moved R10 9.00 mm to (106.0, 83.6)
- moved R7 9.00 mm to (115.0, 83.6)
- moved C8 6.32 mm to (119.7, 110.8), turned to -135 degrees
- moved P1 4.68 mm to (115.5, 104.5)
- moved R16 3.00 mm to (186.0, 83.0)
- moved R17 3.00 mm to (189.0, 83.0)
- moved Q1 0.70 mm to (140.9, 92.8)
Connections:
- Q1 pad 1: Net-(Q1-B) -> Earth
- Q1 pad 2: Net-(BZ1--) -> Net-(Q1-B)
- Q1 pad 3: Earth -> Net-(BZ1--)
